File: 0024_Speaker_Module_PAM8302.kicad_sch (KiCad schematic)
At the start: 12 parts, among them J1 Screw_Terminal_01x02, U1 PAM8302AAY

Commit message: Add files via upload
Parts:
- removed U1: PAM8302AAY, Package_DFN_QFN:DFN-8-1EP_3x3mm_P0.65mm_EP1.55x2.4mm, symbol Amplifier_Audio:PAM8302AAY
- added C5: 10uF, Capacitor_SMD:C_0603_1608Metric, symbol Device:C
- added D1: LED, LED_SMD:LED_0805_2012Metric, symbol Device:LED
- added R4: R, Resistor_SMD:R_0805_2012Metric, symbol Device:R
- added U2: ~, Moduler_:pin_header, symbol moduler_pin:air
- added U3: PAM8302AAS, Package_SO:MSOP-8_3x3mm_P0.65mm, symbol Amplifier_Audio:PAM8302AAS
- C1, C2: footprint (none) -> Capacitor_SMD:C_0805_2012Metric
- C3, C4: value C -> 220pF; footprint (none) -> Capacitor_SMD:C_0805_2012Metric
- FB1, FB2: footprint (none) -> Inductor_SMD:L_0805_2012Metric
- J1: footprint (none) -> TerminalBlock_Phoenix:TerminalBlock_Phoenix_MKDS-1,5-2-5.08_1x02_P5.08mm_Horizontal
- R1, R2, R3: footprint (none) -> Resistor_SMD:R_0805_2012Metric
- RV1: footprint (none) -> memin:3362P_1
Connections:
- net AIN+: now also U2.13
- net AIN-: now also U2.12
- net GND: now also C5.1, D1.1 (K), U2.9, U3.7 (GND)
- net at R2.2: now also U3.4 (IN-)
- net at FB1.1: now also U3.5 (OUT+)
- net SD: now reaches R3.1
- net SD: now also U2.14, U3.1 (~{SD})
- net at R1.2: now also U3.3 (IN+)
- net at FB2.1: now also U3.8 (OUT-)
- net VCC renamed +3V3
- net +3V3: now also C5.2, R4.1, U2.8, U3.6 (VDD)
- new net: D1.2 (A), R4.2
- no-connect marks 0 -> 13
Other:
- note added: "AIR PIN"
- note added: "SENSOR"
- moved on the sheet: C1, C2, C3, C4, FB1, FB2, J1, R1, R2, R3, RV1
